Commit message: IK working

File: moveit_config/config/arm.ros2_control.xacro (robot description, xacro)
@@ -1,5 +1,5 @@
 <?xml version="1.0"?>
 <robot xmlns:xacro="http://www.ros.org/wiki/xacro">
-    <xacro:macro name="urdf_ros2_control" params="name initial_positions_file">
+    <xacro:macro name="arm_ros2_control" params="name initial_positions_file">
         <xacro:property name="initial_positions" value="${xacro.load_yaml(initial_positions_file)['initial_positions']}"/>
         <ros2_control name="${name}" type="system">
@@ -13,4 +13,5 @@
                   <param name="initial_value">${initial_positions['base-l1']}</param>
                 </state_interface>
+                <state_interface name="velocity"/>
             </joint>
             <joint name="l1-l2">
@@ -19,4 +20,5 @@
                   <param name="initial_value">${initial_positions['l1-l2']}</param>
                 </state_interface>
+                <state_interface name="velocity"/>
             </joint>
             <joint name="l2-l3">
@@ -25,4 +27,5 @@
                   <param name="initial_value">${initial_positions['l2-l3']}</param>
                 </state_interface>
+                <state_interface name="velocity"/>
             </joint>
             <joint name="l3-l4">
@@ -31,4 +34,5 @@
                   <param name="initial_value">${initial_positions['l3-l4']}</param>
                 </state_interface>
+                <state_interface name="velocity"/>
             </joint>
             <joint name="l4-l5">
@@ -37,4 +41,5 @@
                   <param name="initial_value">${initial_positions['l4-l5']}</param>
                 </state_interface>
+                <state_interface name="velocity"/>
             </joint>
             <joint name="l5-l6">
@@ -43,4 +48,12 @@
                   <param name="initial_value">${initial_positions['l5-l6']}</param>
                 </state_interface>
+                <state_interface name="velocity"/>
+            </joint>
+            <joint name="l6-hand">
+                <command_interface name="position"/>
+                <state_interface name="position">
+                  <param name="initial_value">${initial_positions['l6-hand']}</param>
+                </state_interface>
+                <state_interface name="velocity"/>
             </joint>
         </ros2_control>
